File: Circuit/MainBoard_V1/MainBoard_V1.kicad_sch (KiCad schematic)
At the start: 0 parts

Commit message: 回路図書いてる途中
Parts:
- added BZ1: Buzzer, Buzzer_Beeper:Buzzer_Murata_PKLCS1212E, symbol Device:Buzzer
- added C1, C11, C12, C13, C17, C18, C22, C9: 0.1uf, Capacitor_SMD:C_0603_1608Metric, symbol Device:C
- added C10: 4.7u, Capacitor_SMD:C_0805_2012Metric, symbol Device:C
- added C2, C4, C6, C7: 10u, Capacitor_SMD:C_0805_2012Metric, symbol Device:C
- added C20: 2200pf, Capacitor_SMD:C_0603_1608Metric, symbol Device:C
- added C3, C31, C5, C8: 100uf, Capacitor_THT:CP_Radial_D5.0mm_P2.00mm, symbol Device:C_Polarized
- added D1, D2, D4: 1N4148W, Diode_SMD:D_SOD-123, symbol Diode:1N4148W
- added D10, D11, D13, D23, D3, D6, D7, D8, D9: LED, LED_SMD:LED_0603_1608Metric, symbol Device:LED
- added D5: CH213K, Package_TO_SOT_SMD:TSOT-23, symbol 0-MyLibrary:CH213K
- added H1, H2, H3, H4: MountingHole, MountingHole:MountingHole_3.2mm_M3_Pad_Via, symbol Mechanical:MountingHole
- added J1, J2, J3, J5: Conn_01x04, Connector_JST:JST_PH_B4B-PH-K_1x04_P2.00mm_Vertical, symbol Connector_Generic:Conn_01x04
- added J4: Conn_01x07, Connector_JST:JST_PH_B7B-PH-K_1x07_P2.00mm_Vertical, symbol Connector_Generic:Conn_01x07
- added J6: Raspberry_Pi_2_3, symbol Connector:Raspberry_Pi_2_3
- added Q1, Q3: Q_PMOS_GDS, Package_TO_SOT_SMD:TO-252-2, symbol Device:Q_PMOS_GDS
- added Q2: BSS138, Package_TO_SOT_SMD:SOT-23, symbol Transistor_FET:BSS138
- added R1, R10, R13, R15, R16, R2, R20, R22, R3, R4, R5, R6: 10k, Resistor_SMD:R_0603_1608Metric, symbol Device:R
- added R11, R12, R14, R17, R18, R21, R30, R7, R8, R9: 1k, Resistor_SMD:R_0603_1608Metric, symbol Device:R
- added R19: 10, Resistor_SMD:R_0603_1608Metric, symbol Device:R
- added R28, R29: 4.7k, Resistor_SMD:R_0603_1608Metric, symbol Device:R
- added SW1, SW2, SW4, SW5: SW_Push, Button_Switch_SMD:SW_SPST_PTS810, symbol Switch:SW_Push
- added SW3, SW6: SW_Slide_DPDT, 0-MyLibrary:IS-2235, symbol Switch:SW_Slide_DPDT
- added TP1, TP2, TP3, TP4, TP5: TestPoint, TestPoint:TestPoint_THTPad_D1.0mm_Drill0.5mm, symbol Connector:TestPoint
- added U2: LM1117MP-3.3, Package_TO_SOT_SMD:SOT-223-3_TabPin2, symbol Regulator_Linear:LM1117MP-3.3
- added U3: STM32F446RETx, Package_QFP:LQFP-64_10x10mm_P0.5mm, symbol MCU_ST_STM32F4:STM32F446RETx
- added U9: MPU-6050, Sensor_Motion:InvenSense_QFN-24_4x4mm_P0.5mm, symbol Sensor_Motion:MPU-6050
- added Y1: CSTNE16M0V530000R0, Crystal:Resonator_SMD_Murata_CSTxExxV-3Pin_3.0x1.1mm, symbol CSTNE16M0V530000R0:CSTNE16M0V530000R0
Connections:
- new net: D6.2 (A), R7.1
- new net: C7.1, D4.2 (A), D5.3 (VI), U2.2 (VO)
- new net: D9.2 (A), R8.1
- new net: D11.2 (A), R10.1
- new net: Q1.1 (G), R1.2, SW3.1 (A), SW3.6 (C)
- new net: Q3.1 (G), R15.2, SW6.1 (A), SW6.6 (C)
- new net: Q2.1 (G), R19.2, R20.2
- new net: C10.1, U3.30 (VCAP_1)
- new net: D3.2 (A), R22.1
- new net: D8.2 (A), R12.1
- new net: BZ1.2 (-), Q2.3 (D), R18.1
- new net: D13.2 (A), R17.1
- new net: D7.2 (A), R11.1
- new net: D10.2 (A), R9.1
- new net: D23.2 (A), R30.1
- new net: C20.1, U9.20 (CPOUT)
- new net: R4.2, U3.60 (BOOT0)
- new net: C22.1, U9.10 (REGOUT)
- new net: U3.5 (PH0), Y1.1
- new net: U3.6 (PH1), Y1.3
- new net: J6.1 (3V3), J6.17 (3V3)
- new net +3V3: C11.2, C12.2, C13.2, C17.1, C18.2, C9.2, D5.2 (VO), J1.2 (Pin_2), J2.2 (Pin_2), J3.2 (Pin_2), J4.2 (Pin_2), J5.2 (Pin_2), R28.1, R29.1, R3.2, R8.2, SW1.2, SW4.2, SW5.2, TP4.1, U3.1 (VBAT), U3.13 (VDDA), U3.19 (VDD), U3.32 (VDD), U3.48 (VDD), U3.64 (VDD), U9.13 (VDD), U9.8 (VLOGIC)
- new net +5V: C6.2, D4.1 (K), J6.2 (5V), J6.4 (5V), R9.2, TP5.1, U2.3 (VI)
- new net +BATT: D1.1 (K), Q3.3 (S), R15.1
- new net +BATTP: D2.1 (K), Q1.3 (S), R1.1
- new net BTN1: R2.1, SW1.1
- new net BTN2: R5.1, SW4.1
- new net BTN3: R6.1, SW5.1
- new net BUZZER: R19.1
- new net GND: C1.1, C10.2, C11.1, C12.1, C13.1, C2.2, C20.2, C22.2, C3.2, C6.1, C7.2, C8.2, C9.1, D10.1 (K), D11.1 (K), D13.1 (K), D23.1 (K), D5.1 (GND), D6.1 (K), D7.1 (K), D8.1 (K), D9.1 (K), J1.1 (Pin_1), J2.1 (Pin_1), J3.1 (Pin_1), J4.1 (Pin_1), J5.1 (Pin_1), J6.14 (GND), J6.20 (GND), J6.25 (GND), J6.30 (GND), J6.34 (GND), J6.39 (GND), J6.6 (GND), J6.9 (GND), Q2.2 (S), R14.1, R2.2, R20.1, R4.1, R5.2, R6.2, SW2.1, SW6.2 (B), SW6.5 (B), TP3.1, U2.1 (GND), U3.12 (VSSA), U3.18 (VSS), U3.31 (VSS), U3.47 (VSS), U3.63 (VSS), U9.1 (CLKIN), U9.11 (FSYNC), U9.18 (GND), U9.9 (AD0), Y1.2
- new net GND1: C17.2, C18.1
- new net GND2: R21.1
- new net GNDP: C31.2, C4.2, C5.2, D3.1 (K), SW3.2 (B), SW3.5 (B)
- new net NRST: C1.2, J4.5 (Pin_5), R3.1, SW2.2, U3.7 (NRST)
- new net PC_RX: J4.7 (Pin_7)
- new net PC_TX: J4.6 (Pin_6)
- new net RAS_RX: J6.10 (GPIO15/RXD)
- new net RAS_TX  : J6.8 (GPIO14/TXD)
- new net RX1: J1.4 (Pin_4)
- new net RX2: J2.4 (Pin_4)
- new net RX3: J3.4 (Pin_4)
- new net SCL: R29.2, TP2.1, U9.23 (SCL)
- new net SDA: R28.2, TP1.1, U9.24 (SDA)
- new net STM_LED1: R7.2
- new net STM_LED2: R11.2
- new net STM_LED3: R12.2
- new net STM_LED4: R17.2
- new net SWCLK: J4.4 (Pin_4), U3.49 (PA14)
- new net SWDIO: J4.3 (Pin_3), U3.46 (PA13)
- new net TX1: J1.3 (Pin_3)
- new net TX2: J2.3 (Pin_3)
- new net TX3: J3.3 (Pin_3)
- new net VBUS: R30.2
- new net VCC: BZ1.1 (+), C2.1, C3.1, C8.1, D1.2 (A), Q3.2 (D), R10.2, R13.2, R18.2
- new net VCC2: R16.2
- new net VCCP: C31.1, C4.1, C5.1, D2.2 (A), Q1.2 (D), R22.2
- new net VOLTAGE1: R13.1, R14.2, R16.1, R21.2
Other:
- note added: "MPU6050"
- note added: "Mounting hole"
- note added: "STM32 F446RE"

Commit message: 進捗
Parts:
- removed D23: LED, LED_SMD:LED_0603_1608Metric, symbol Device:LED
- removed J1: Conn_01x04, Connector_JST:JST_PH_B4B-PH-K_1x04_P2.00mm_Vertical, symbol Connector_Generic:Conn_01x04
- removed R30: 1k, Resistor_SMD:R_0603_1608Metric, symbol Device:R
- added C3, C?: 10u, Capacitor_SMD:C_0805_2012Metric, symbol Device:C
- added D1: 1N4148W, Diode_SMD:D_SOD-123, symbol Diode:1N4148W
- added F1, F2: Fuse, Fuse:Fuseholder_Clip-5x20mm_Keystone_3517_Inline_P23.11x6.76mm_D1.70mm_Horizontal, symbol Device:Fuse
- added J10, J11, J12, J6, J7, J8, J9: Conn_01x04, Connector_JST:JST_XH_B4B-XH-A_1x04_P2.50mm_Vertical, symbol Connector_Generic:Conn_01x04
- added U11: LM78M05_TO252, Package_TO_SOT_SMD:TO-252-2, symbol Regulator_Linear:LM78M05_TO252
- J2: renamed from J6; footprint (none) -> 0-MyLibrary:raspberreyPi_2_3
- J3: renamed from J2; footprint Connector_JST:JST_PH_B4B-PH-K_1x04_P2.00mm_Vertical -> Connector_JST:JST_XH_B4B-XH-A_1x04_P2.50mm_Vertical
- J4: renamed from J3; footprint Connector_JST:JST_PH_B4B-PH-K_1x04_P2.00mm_Vertical -> Connector_JST:JST_XH_B4B-XH-A_1x04_P2.50mm_Vertical
- J5: footprint Connector_JST:JST_PH_B4B-PH-K_1x04_P2.00mm_Vertical -> Connector_JST:JST_XH_B4B-XH-A_1x04_P2.50mm_Vertical
- renumbered C2 to C1, C9 to C10, C17 to C11, C18 to C12, C10 to C13, C11 to C14, C12 to C15, C13 to C16, C20 to C17, C22 to C18, C4 to C2, C6 to C3, C7 to C4, C1 to C5, C3 to C6, C5 to C7, C31 to C9, D4 to D1, D8 to D12, D1 to D2, D2 to D3, D5 to D4, D11 to D5, D3 to D6, D6 to D7, D7 to D8, J4 to J1, Q3 to Q1, Q1 to Q2, Q2 to Q3, R15 to R1, R13 to R10, R14 to R11, R16 to R12, R21 to R13, R7 to R14, R8 to R15, R9 to R16, R11 to R18, R12 to R19, R1 to R2, R17 to R20, R18 to R21, R19 to R22, R20 to R23, R28 to R24, R29 to R25, R2 to R4, R4 to R5, R5 to R6, R6 to R7, R10 to R8, R22 to R9, SW2 to SW1, SW1 to SW2, SW6 to SW3, SW3 to SW4, SW4 to SW5, SW5 to SW6, TP5 to TP3, TP3 to TP5, U2 to U1, U3 to U2, U9 to U3
Connections:
- net VCC2 is gone; now on net VCCP: R12.2
- net +3V3: now also J10.2 (Pin_2), J11.2 (Pin_2), J12.2 (Pin_2), J6.2 (Pin_2), J7.2 (Pin_2), J8.2 (Pin_2), J9.2 (Pin_2); no longer J3.2 (Pin_2), J4.2 (Pin_2), J5.2 (Pin_2)
- net +5V: now also C3.1, D1.2 (A), U11.3 (VO)
- net +BATT: now also F1.1; no longer D2.1 (K), Q1.3 (S), R1.1
- net +BATTP: now also F2.1; no longer D3.1 (K), Q2.3 (S), R2.1
- net GND: now also C3.2, C?.1, J10.1 (Pin_1), J11.1 (Pin_1), J12.1 (Pin_1), J6.1 (Pin_1), J7.1 (Pin_1), J8.1 (Pin_1), J9.1 (Pin_1), U11.2 (GND)
- net RX1: now also U2.43 (PA10)
- net RX2: now also U2.17 (PA3)
- net RX3: now also U2.52 (PC11)
- net TX1: now also U2.42 (PA9)
- net TX2: now also U2.16 (PA2)
- net TX3: now also U2.51 (PC10)
- net VCC: now also C?.2, D1.1 (K), U11.1 (VI)
- net VCCP: now also J3.2 (Pin_2), J4.2 (Pin_2), J5.2 (Pin_2)
- net TX4: now reaches J5.3 (Pin_3)
- net TX4: now also U2.14 (PA0)
- net RX4: now reaches J5.4 (Pin_4)
- net RX4: now also U2.15 (PA1)
- net TX6: now reaches U2.37 (PC6)
- net RX6: now reaches U2.38 (PC7)
- net TX5: now reaches U2.53 (PC12)
- net TX5: now also J6.3 (Pin_3)
- net RX5: now reaches U2.54 (PD2)
- net RX5: now also J6.4 (Pin_4)
- new net: D2.1 (K), F1.2, Q1.3 (S), R1.1
- new net: D3.1 (K), F2.2, Q2.3 (S), R2.1
- new net ECHO1: J7.4 (Pin_4)
- new net ECHO2: J8.4 (Pin_4)
- new net ECHO3: J9.4 (Pin_4)
- new net ECHO4: J10.4 (Pin_4)
- new net ECHO5: J11.4 (Pin_4)
- new net ECHO6: J12.4 (Pin_4)
- new net TRIG1: J7.3 (Pin_3)
- new net TRIG2: J8.3 (Pin_3)
- new net TRIG3: J9.3 (Pin_3)
- new net TRIG4: J10.3 (Pin_3)
- new net TRIG5: J11.3 (Pin_3)
- new net TRIG6: J12.3 (Pin_3)
Other:
- moved on the sheet: C1, C2, C6, C7, C8, C9, D2, D3, J5, Q1, Q2, R1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

Commit message: 配線と配置を進めた
Parts:
- removed C8, C9: 100uf, Capacitor_THT:CP_Radial_D5.0mm_P2.00mm, symbol Device:C_Polarized
- removed U11: LM78M05_TO252, Package_TO_SOT_SMD:TO-252-2, symbol Regulator_Linear:LM78M05_TO252
- added J10, J14: Conn_01x04, Connector_JST:JST_XH_B4B-XH-A_1x04_P2.50mm_Vertical, symbol Connector_Generic:Conn_01x04
- added MD1: OKL-T_6-W12N-C, 0-MyLibrary:MURATA_OKL-T-6-W12N-C_0, symbol OKL-T_6-W12N-C:OKL-T_6-W12N-C
- added R4: 10k, Resistor_SMD:R_0603_1608Metric, symbol Device:R
- added R8: 1k, Resistor_SMD:R_0603_1608Metric, symbol Device:R
- added R9: 330, Resistor_SMD:R_0603_1608Metric, symbol Device:R
- added TP1, TP2, TP3, TP4: TestPoint, TestPoint:TestPoint_THTPad_D4.0mm_Drill2.0mm, symbol Connector:TestPoint
- gave numbers to parts that had none: 1
- renumbered C5 to C1, C13 to C11, C14 to C12, C15 to C13, C16 to C14, C11 to C15, C12 to C16, C1 to C4, C2 to C5, C3 to C8, C4 to C9, D9 to D10, D10 to D11, D5 to D12, D6 to D13, D7 to D4, D8 to D5, D1 to D6, D12 to D7, D4 to D8, D13 to D9, J10 to J11, J11 to J12, J12 to J13, J3 to J2, J4 to J3, J5 to J4, J6 to J5, J2 to J6, R3 to R1, R7 to R10, R14 to R11, R18 to R12, R19 to R13, R15 to R14, R16 to R15, R8 to R16, R9 to R17, R10 to R18, R11 to R19, R4 to R2, R12 to R20, R13 to R21, R20 to R22, R21 to R23, R22 to R24, R23 to R25, R24 to R26, R25 to R27, R5 to R3, R6 to R5, R1 to R6, R2 to R7, SW5 to SW3, SW3 to SW4, SW4 to SW5, TP1 to TP5, TP2 to TP6, TP3 to TP7, TP4 to TP8, TP5 to TP9, U2 to U1, U1 to U2
Connections:
- net GND1 is gone; now on net GND: C15.2, C16.1
- net +3V3: now also J10.2 (Pin_2), J14.2 (Pin_2)
- net +5V: now also MD1.4 (VOUT)
- net +BATT: now also TP1.1
- net +BATTP: now also TP2.1
- net GND: now also J10.1 (Pin_1), J14.1 (Pin_1), MD1.3 (1_GROUND), MD1.7 (2_GROUND), R9.1, TP3.1
- net GNDP: now also TP4.1
- net VCC: now also MD1.2 (VIN), R4.1
- net VOLTAGE1 renamed VOLTAGE
- net VOLTAGE: no longer R20.1, R21.2
- new net: MD1.1 (~{ON}/OFF_CONTROL), R4.2
- new net: R8.1, R9.2
- new net: MD1.6 (TRIM), R8.2
- new net ECHO7: J10.4 (Pin_4)
- new net ECHO8: J14.4 (Pin_4)
- new net TRIG7: J10.3 (Pin_3)
- new net TRIG8: J14.3 (Pin_3)
- new net VOLTAGEP: R20.1, R21.2
Other:
- note added: "Connectors"
- note added: "RasPi"
- note added: "Supply"
- moved on the sheet: BZ1, C1, C10, C11, C12, C13, C14, C15, C16, C17, C18, C2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
