File: Circuit/MainBoard_V1/MainBoard_V1.kicad_sch (KiCad schematic)
At the start: 118 parts, among them J1 Conn_01x07, J10 Conn_01x04, J11 Conn_01x04, J12 Conn_01x04, J13 Conn_01x04, J14 Conn_01x04, J15 Conn_01x02, J2 Conn_01x04, J3 Conn_01x04, J4 Conn_01x04, J5 Conn_01x04, J6 Raspberry_Pi_2_3, J7 Conn_01x04, J8 Conn_01x04, J9 Conn_01x04, Q1 Q_PMOS_GDS, Q2 Q_PMOS_GDS, Q3 BSS138, Q4 BSS138, Q5 BSS138, Q6 BSS138, Q7 BSS138, SW1 SW_Push, SW2 SW_Push, SW3 SW_Push, SW4 SW_Slide_DPDT, SW5 SW_Slide_DPDT, SW6 SW_Push, U1 STM32F446RETx, U2 LM1117MP-3.3, U3 MPU-6050, Y1 CSTNE16M0V530000R0

Commit message: 配線進捗
Parts:
- removed J13, J14: Conn_01x04, Connector_JST:JST_XH_B4B-XH-A_1x04_P2.50mm_Vertical, symbol Connector_Generic:Conn_01x04
- gave numbers to parts that had none: 3
- renumbered J15 to J13
Connections:
- net RX1 is gone; now on net PC_TX: U1.43 (PA10)
- net RX6 is gone; now on net RAS_TX  : U1.38 (PC7)
- net TX1 is gone; now on net PC_RX: U1.42 (PA9)
- net TX6 is gone; now on net RAS_RX: U1.37 (PC6)
- net ECHO1: now also J7.3 (Pin_3), U1.45 (PA12); no longer J7.4 (Pin_4)
- net ECHO2: now also J8.3 (Pin_3), U1.41 (PA8); no longer J8.4 (Pin_4)
- net ECHO3: now also J9.3 (Pin_3), U1.40 (PC9); no longer J9.4 (Pin_4)
- net ECHO4: now also J10.3 (Pin_3), U1.36 (PB15); no longer J10.4 (Pin_4)
- net ECHO5: now also J11.3 (Pin_3), U1.34 (PB13); no longer J11.4 (Pin_4)
- net ECHO6: now also J12.3 (Pin_3), U1.29 (PB10); no longer J12.4 (Pin_4)
- net LED1_SIG: now also U1.27 (PB1)
- net LED2_SIG: now also U1.26 (PB0)
- net LED3_SIG: now also U1.23 (PA7)
- net LED4_SIG: now also U1.22 (PA6)
- net RX3: now also J5.4 (Pin_4); no longer J3.4 (Pin_4)
- net RX4: now also J3.4 (Pin_4); no longer J4.4 (Pin_4)
- net RX5: now also J4.4 (Pin_4); no longer J5.4 (Pin_4)
- net TRIG1: now also J7.4 (Pin_4), U1.50 (PA15); no longer J7.3 (Pin_3)
- net TRIG2: now also J8.4 (Pin_4), U1.44 (PA11); no longer J8.3 (Pin_3)
- net TRIG3: now also J9.4 (Pin_4), U1.39 (PC8); no longer J9.3 (Pin_3)
- net TRIG4: now also J10.4 (Pin_4), U1.35 (PB14); no longer J10.3 (Pin_3)
- net TRIG5: now also J11.4 (Pin_4), U1.33 (PB12); no longer J11.3 (Pin_3)
- net TRIG6: now also J12.4 (Pin_4), U1.28 (PB2); no longer J12.3 (Pin_3)
- net TX3: now also J5.3 (Pin_3); no longer J3.3 (Pin_3)
- net TX4: now also J3.3 (Pin_3); no longer J4.3 (Pin_3)
- net TX5: now also J4.3 (Pin_3); no longer J5.3 (Pin_3)

Commit message: 進捗
Parts:
- removed J12, J2, J3, J5: Conn_01x04, Connector_JST:JST_XH_B4B-XH-A_1x04_P2.50mm_Vertical, symbol Connector_Generic:Conn_01x04
- removed R10: 10k, Resistor_SMD:R_0603_1608Metric, symbol Device:R
- removed SW6: SW_Push, Button_Switch_SMD:SW_SPST_PTS810, symbol Switch:SW_Push
- added J1, J2, J3: Conn_01x02, Connector_JST:JST_PH_B2B-PH-K_1x02_P2.00mm_Vertical, symbol Connector_Generic:Conn_01x02
- added J10, J11, J12: Conn_01x03, Connector_JST:JST_XH_B3B-XH-A_1x03_P2.50mm_Vertical, symbol Connector_Generic:Conn_01x03
- added J5, J6, J7: Conn_01x02, Connector_JST:JST_XH_B2B-XH-A_1x02_P2.50mm_Vertical, symbol Connector_Generic:Conn_01x02
- renumbered J7 to J13, J8 to J14, J9 to J15, J10 to J16, J11 to J17, J13 to J18, J14 to J19, J15 to J20, J16 to J21, J1 to J8, J6 to J9
Connections:
- net +3V3: now also J10.2 (Pin_2), J11.2 (Pin_2), J12.2 (Pin_2)
- net +5V: now also J4.2 (Pin_2)
- net BTN1: now also U1.3 (PC14)
- net BTN2: now also U1.2 (PC13)
- net GND: now also J10.1 (Pin_1), J11.1 (Pin_1), J12.1 (Pin_1)
- net GNDP: now also J5.1 (Pin_1), J6.1 (Pin_1), J7.1 (Pin_1)
- net RX2: now also J1.2 (Pin_2)
- net RX3: now also J4.4 (Pin_4)
- net RX4: now also J2.2 (Pin_2)
- net RX5: now also J3.2 (Pin_2); no longer J4.4 (Pin_4)
- net SCL: now also U1.61 (PB8)
- net SDA: now also U1.62 (PB9)
- net STM_LED1: now also U1.56 (PB4)
- net STM_LED2: now also U1.57 (PB5)
- net STM_LED3: now also U1.58 (PB6)
- net STM_LED4: now also U1.59 (PB7)
- net TX2: now also J1.1 (Pin_1)
- net TX3: now also J4.3 (Pin_3)
- net TX4: now also J2.1 (Pin_1)
- net TX5: now also J3.1 (Pin_1); no longer J4.3 (Pin_3)
- net VCCP: now also J5.2 (Pin_2), J6.2 (Pin_2), J7.2 (Pin_2); no longer J4.2 (Pin_2)
- net ADC3: now reaches U1.20 (PA4)
- net ADC3: now also J12.3 (Pin_3)
- net ADC2: now reaches U1.21 (PA5)
- net ADC2: now also J11.3 (Pin_3)
- net ADC1: now reaches U1.24 (PC4)
- net ADC1: now also J10.3 (Pin_3)
- net ECHO6: no longer names the net of U1.29 (PB10)
- net TRIG6: no longer names the net of U1.28 (PB2)
Other:
- moved on the sheet: J13, J14, J15, J16, J17, J18, J19, J20, J21, J8
