File: Circuit/MainBoard_V1/_autosave-MainBoard_V1.kicad_pcb (KiCad board)
At the start: 2 copper layers, 56 x 65 mm, 122 parts, among them J1 Conn_01x02, J10 Conn_01x03, J11 Conn_01x03, J12 Conn_01x03, J13 Conn_01x04, J14 Conn_01x04, J15 Conn_01x04, J16 Conn_01x04, J17 Conn_01x04, J18 Conn_01x02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

Commit message: ほぼ完成
Routing:
- net GND: vias 198 -> 215
Other:
- board text added: "SIG"
- board text added: "STM32 F446RE"
