File: Circuit/MainBoard_V1/MainBoard_V1.kicad_pcb (KiCad board)
At the start: 2 copper layers, 56 x 65 mm, 122 parts, among them J1 Conn_01x02, J10 Conn_01x03, J11 Conn_01x03, J12 Conn_01x03, J13 Conn_01x04, J14 Conn_01x04, J15 Conn_01x04, J16 Conn_01x04, J17 Conn_01x04, J18 Conn_01x02, J19 Conn_01x02, J2 Conn_01x02, J20 Conn_01x02, J21 Conn_01x02, J3 Conn_01x02, J4 Conn_01x04, J5 Conn_01x02, J6 Conn_01x02, J7 Conn_01x02, J8 Conn_01x07, J9 Raspberry_Pi_2_3, Q1 Q_PMOS_GDS, Q2 Q_PMOS_GDS, Q3 BSS138, Q4 BSS138, Q5 BSS138, Q6 BSS138, Q7 BSS138, SW1 SW_Push, SW2 SW_Push, SW3 SW_Push, SW4 SW_Slide_DPDT, SW5 SW_Slide_DPDT, U1 STM32F446RETx, U2 LM1117MP-3.3, U3 MPU-6050, Y1 CSTNE16M0V530000R0

Commit message: 発注データ
Routing:
- net GND: vias 198 -> 216
Other:
- board text added: "MPU6050"
- board text added: "MainBoard V1"
- board text added: "P"
- board text added: "PULL UP"
- board text added: "S"
- board text added: "SIG"
- board text added: "STM32 F446RE"
- board text added: "VCC-P"
- board text added: "VCC-S"

Commit message: 多分何も変わってないけど一応
Other:
- board text added: "ADC"
- board text added: "BUZZER"
- board text added: "DCDC"
- board text added: "FUZE"
- board text added: "GPIO"
- board text added: "LED"
- board text added: "POWER"
- board text added: "SIGNAL"
- board text added: "STM"
- board text removed: "VCC"
