File: Circuit/MainBoard_V3/_autosave-MainBoard_V3.kicad_pcb (KiCad board)
At the start: 2 copper layers, 56 x 65 mm, 134 parts, among them J1 Conn_01x02, J10 Conn_01x03, J11 Conn_01x03, J12 Conn_01x04, J13 Conn_01x04, J14 Conn_01x04, J15 Conn_01x04, J2 Conn_01x02, J3 Conn_01x02, J4 Conn_01x04, J5 Conn_01x02, J6 Conn_01x02, J7 Conn_01x02, J8 Conn_01x07, J9 Raspberry_Pi_2_3, Q1 Q_PMOS_GDS, Q10 BSS138, Q2 Q_PMOS_GDS, Q3 BSS138, Q4 IRLML6402, Q5 BSS138, Q6 BSS138, Q7 BSS138, Q8 BSS138, Q9 BSS138, SW1 SW_Push, SW2 SW_Push, SW3 SW_Push, SW4 SW_Slide_DPDT, SW5 SW_Slide_DPDT, U1 STM32F446RETx, U2 LM1117MP-3.3, U3 MPU-6050, Y1 CSTNE16M0V530000R0

Commit message: 回路図と配置と配線が半分ほど終わり
Parts:
- moved R19 4.03 mm to (145.2, 112.8), turned to -90 degrees
- moved R20 3.04 mm to (141.8, 112.8), turned to 90 degrees
- moved C13 2.57 mm to (143.5, 112.8), turned to 90 degrees
Routing:
- net +3V3: track 10.5 -> 41.7 mm
- net RX2: track 61.4 -> 73.1 mm
- net TX2: track 55.8 -> 67.5 mm
- net RX5: track 10.6 -> 16.1 mm
- net ECHO1: track 7.41 -> 12.7 mm
- net TRIG1: track 8.24 -> 13.5 mm
- net PC_RX: track 40.6 -> 45.6 mm
- net PC_TX: track 37.3 -> 41.8 mm
- net NRST: track 34.2 -> 38.7 mm
- net SWCLK: track 31.1 -> 35.6 mm
- net SWDIO: track 28.3 -> 32.6 mm
- net TX4: track 30.7 -> 34.8 mm
- net ECHO2: track 12.6 -> 16.3 mm
- net RX4: track 28.2 -> 31.7 mm
- net TRIG2: track 14.7 -> 18.2 mm
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