File: Circuit/MainBoard_V3/MainBoard_V3.kicad_pcb (KiCad board)
At the start: 2 copper layers, 56 x 65 mm, 134 parts, among them J1 Conn_01x02, J10 Conn_01x03, J11 Conn_01x03, J12 Conn_01x04, J13 Conn_01x04, J14 Conn_01x04, J15 Conn_01x04, J2 Conn_01x02, J3 Conn_01x02, J4 Conn_01x04, J5 Conn_01x02, J6 Conn_01x02, J7 Conn_01x02, J8 Conn_01x07, J9 Raspberry_Pi_2_3, Q1 Q_PMOS_GDS, Q10 BSS138, Q2 Q_PMOS_GDS, Q3 BSS138, Q4 IRLML6402, Q5 BSS138, Q6 BSS138, Q7 BSS138, Q8 BSS138, Q9 BSS138, SW1 SW_Push, SW2 SW_Push, SW3 SW_Push, SW4 SW_Slide_DPDT, SW5 SW_Slide_DPDT, U1 STM32F446RETx, U2 LM1117MP-3.3, U3 MPU-6050, Y1 CSTNE16M0V530000R0

Commit message: 進捗
Parts:
- moved C8 4.78 mm to (129.6, 171.2)
- moved R19 4.03 mm to (145.2, 112.8), turned to -90 degrees
- moved R20 3.04 mm to (141.8, 112.8), turned to 90 degrees
- moved C13 2.57 mm to (143.5, 112.8), turned to 90 degrees
Routing:
- net +3V3: track 10.5 -> 41.7 mm
- net RX2: track 61.4 -> 73.1 mm
- net TX2: track 55.8 -> 67.5 mm
- net RX5: track 10.6 -> 16.1 mm
- net ECHO1: track 7.41 -> 12.7 mm
- net TRIG1: track 8.24 -> 13.5 mm
- net PC_RX: track 40.6 -> 45.6 mm
- net PC_TX: track 37.3 -> 41.8 mm
- net NRST: track 34.2 -> 38.7 mm
- net SWCLK: track 31.1 -> 35.6 mm
- net SWDIO: track 28.3 -> 32.6 mm
- net TX4: track 30.7 -> 34.8 mm
- net ECHO2: track 12.6 -> 16.3 mm
- net RX4: track 28.2 -> 31.7 mm
- net TRIG2: track 14.7 -> 18.2 mm
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
Commit message: 大体設計終わり あとGNDビア
Parts:
- removed R28: 1k, Resistor_SMD:R_0603_1608Metric
- removed TP5, TP6, TP7: TestPoint, TestPoint:TestPoint_THTPad_D1.0mm_Drill0.5mm
- added C28: 100uf, Capacitor_THT:CP_Radial_D6.3mm_P2.50mm, F.Cu at (10.3, -19.8)
- added C29: 100uf, Capacitor_THT:CP_Radial_D6.3mm_P2.50mm, F.Cu at (3.25, -19.8)
- BZ1, C11, C4, C9, Q6, R1, R26, R29, R30, R39, R40: moved to B.Cu
- C8: value 100uf -> 10u; footprint Capacitor_THT:CP_Radial_D6.3mm_P2.50mm -> Capacitor_SMD:C_0805_2012Metric
- moved NT1 205.7 mm to (17.5, 2.25)
- moved R19 198.1 mm to (-2.75, -19.0), turned to 0 degrees
- moved C8 197.2 mm to (1.00, 21.7), turned to 180 degrees
- moved J1 194.2 mm to (21.5, 8.75)
- moved J2 194.2 mm to (21.5, -4.75)
- moved J5 194.2 mm to (21.3, 2.25)
- moved J6 194.2 mm to (21.3, -11.3)
- moved R26 193.9 mm to (-2.75, -17.3)
- moved R35 193.4 mm to (-1.25, -29.3), turned to -90 degrees
- moved C13 193.4 mm to (-2.75, -13.8), turned to 180 degrees
- moved R20 193.2 mm to (-2.75, -15.5), turned to 180 degrees
- moved D13 191.5 mm to (-2.75, -17.3), turned to 180 degrees
- moved Q9 189.9 mm to (3.50, -29.3)
- moved R36 189.9 mm to (0.50, -29.3)
- moved R22 188.6 mm to (-8.50, 1.75), turned to 90 degrees
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Connections:
- net ADC2 renamed ENCODER_RIGHT
- J1 pad 1: TX2 -> RX2
- J1 pad 2: RX2 -> TX2
- J10 pad 3: ADC1 -> ENCODER_LEFT
- J2 pad 1: TX4 -> RX4
- J2 pad 2: RX4 -> TX4
- J3 pad 1: TX5 -> RX3
- J3 pad 2: RX5 -> TX3
- J4 pad 4: RX3 -> RX6
- U1 pad 10: VOLTAGEP -> VOLTAGE
- U1 pad 11: VOLTAGE -> VOLTAGEP
- U1 pad 2: BTN2 -> unconnected-(U1-PC13-Pad2)
- U1 pad 20: ADC3 -> ENCODER_LEFT
- U1 pad 22: RW_LED_SIG -> HEAD_LED_SIG
- U1 pad 24: ADC1 -> LIDAR_5V_SIG
- U1 pad 27: HEAD_LED_SIG -> RW_LED_SIG
- U1 pad 29: unconnected-(U1-PB10-Pad29) -> BUZZER
- U1 pad 3: BTN1 -> unconnected-(U1-PC14-Pad3)
- U1 pad 33: TRIG5 -> unconnected-(U1-PB12-Pad33)
- U1 pad 34: ECHO5 -> BTN2
- U1 pad 35: TRIG4 -> BTN1
- U1 pad 36: ECHO4 -> POWER_SIG
- U1 pad 37: RAS_RX -> TX6
- U1 pad 38: RAS_TX -> RX6
- U1 pad 39: TRIG3 -> TRIG2
- U1 pad 40: ECHO3 -> ECHO2
- U1 pad 41: ECHO2 -> LIDAR_OUT
- U1 pad 42: PC_RX -> RAS_RX
- U1 pad 43: PC_TX -> RAS_TX
- U1 pad 44: LIDAR_OUT -> TRIG1
- U1 pad 45: TRIG2 -> ECHO1
- U1 pad 50: ECHO1 -> unconnected-(U1-PA15-Pad50)
- U1 pad 51: TRIG1 -> TX3
- U1 pad 53: TX5 -> PC_RX
- U1 pad 54: RX5 -> PC_TX
- U1 pad 55: BUZZER -> unconnected-(U1-PB3-Pad55)
Routing:
- net +3V3: track 41.7 -> 207.4 mm, vias 0 -> 7
- net TX3: track 0.00 -> 80.0 mm, vias 0 -> 1
- net RX3: track 0.00 -> 74.7 mm, vias 0 -> 1
- net BUZZER: track 0.00 -> 47.1 mm, vias 0 -> 2
- net RW_LED_SIG: track 0.00 -> 45.9 mm, vias 0 -> 1
- net ENCODER_LEFT: track 0.00 -> 37.3 mm
- net BRAKE_LED_SIG: track 0.00 -> 36.8 mm, vias 0 -> 1
- net NRST: track 38.7 -> 74.7 mm, vias 0 -> 6
- net GNDP: track 0.00 -> 33.8 mm, vias 0 -> 16
- net ENCODER_RIGHT: track 0.00 -> 30.7 mm
- net RAS_RX: track 0.00 -> 29.2 mm
- net RAS_TX: track 0.00 -> 28.6 mm
- net TRIG2: track 18.2 -> 46.1 mm, vias 0 -> 1
- net BTN2: track 0.00 -> 27.8 mm, vias 0 -> 2
- net LW_LED_SIG: track 0.00 -> 27.5 mm, vias 0 -> 1
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- added copper zone on B.Cu, net GND
- added copper zone on F.Cu, net GND

Commit message: 電流センスの追加と設計大体終わり
Parts:
- added R28: 5m, Resistor_SMD:R_1206_3216Metric, B.Cu at (10.2, 5.75)
- added R3: 10m, Resistor_SMD:R_1206_3216Metric, B.Cu at (3.00, 5.75)
- added U4: INA180A2, Package_TO_SOT_SMD:SOT-23-5, F.Cu at (2.00, -1.75)
- added U5: INA180A2, Package_TO_SOT_SMD:SOT-23-5, F.Cu at (9.25, -1.75)
- moved R23 5.35 mm to (-9.25, 12.5), turned to 90 degrees
- moved R24 5.06 mm to (-5.75, 12.5), turned to 90 degrees
- moved D11 3.05 mm to (-5.75, 15.8), turned to 90 degrees
- moved R25 2.92 mm to (-7.50, 12.5), turned to 90 degrees
- moved D12 1.90 mm to (-7.50, 15.8), turned to 90 degrees
- moved D10 1.00 mm to (-9.25, 15.8), turned to 90 degrees
- moved C5 0.25 mm to (0.50, 12.2)
- moved NT1 0.25 mm to (17.5, 2.00)
Connections:
- F1 pad 2: Net-(D2-K) -> Net-(U4-+)
- F2 pad 2: Net-(D3-K) -> Net-(U5-+)
- U1 pad 8: unconnected-(U1-PC0-Pad8) -> SENSE_P
- U1 pad 9: unconnected-(U1-PC1-Pad9) -> SENSE
Routing:
- net SENSE_P: track 0.00 -> 23.8 mm, vias 0 -> 2
- net +3V3: track 207.4 -> 223.8 mm, vias 7 -> 9
- net SENSE: track 0.00 -> 14.3 mm, vias 0 -> 2
- net Net-(U5-+): track 0.00 -> 9.83 mm
- net Net-(U4-+): track 0.00 -> 9.83 mm
- net +5V: track 13.4 -> 21.8 mm, vias 19 -> 30
- net Net-(D3-K): track 0.00 -> 5.80 mm, vias 0 -> 1
- net Net-(D2-K): track 0.00 -> 5.80 mm, vias 0 -> 1
- net VCC: track 25.5 -> 27.4 mm
- net BTN2: track 27.8 -> 27.7 mm, vias 2 -> 3
- net GND: vias 160 -> 226
- net BTN1: vias 2 -> 3
Other:
- board text added: "1"
- board text added: "2"
- board text added: "3"
- board text added: "3V3"
- board text added: "4"
- board text added: "5V"
- board text added: "VCC"

Commit message: 完成&製造ファイル生成
Parts:
- added C30: 10u, Capacitor_SMD:C_0805_2012Metric, F.Cu at (-1.00, 13.8)
- added C31: 10u, Capacitor_SMD:C_0805_2012Metric, F.Cu at (-2.75, 21.8)
- added C32: 10u, Capacitor_SMD:C_0805_2012Metric, B.Cu at (-19.8, 22.0)
Connections:
- MD1 pad 10: unconnected-(MD1-POWER_GOOD_OUT-Pad10) -> PGO
Routing:
- net GND: vias 226 -> 227
Other:
- board text added: "+"
- board text added: "-"
- board text added: "LiDAR"
- board text added: "MainBoard V3"
- board text added: "P"
- board text added: "PWR"
- board text added: "RAS"
- board text added: "RST"
- board text added: "RX"
- board text added: "S"
- board text added: "SIG"
- board text added: "STM"
- board text added: "STM32 F446RE"
- board text added: "TX"
- board text added: "VCCP"

Commit message: 製造ファイル再生成
Connections:
- MD1 pad 10: PGO -> unconnected-(MD1-POWER_GOOD_OUT-Pad10)
Changed lines of the file:
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@@
 	(net 76 "unconnected-(MD1-2_NC-Pad9)")
 	(net 77 "Net-(MD1-TRIM)")
-	(net 78 "PGO")
+	(net 78 "unconnected-(MD1-POWER_GOOD_OUT-Pad10)")
 	(net 79 "unconnected-(MD1-1_NC-Pad8)")
 	(net 80 "unconnected-(MD1-4_NC-Pad12)")
@@
 			(size 2.9995 1.143)
 			(layers "F.Cu" "F.Mask" "F.Paste")
-			(net 78 "PGO")
+			(net 78 "unconnected-(MD1-POWER_GOOD_OUT-Pad10)")
 			(pinfunction "POWER_GOOD_OUT")
-			(pintype "open_collector")
+			(pintype "open_collector+no_connect")
 			(solder_mask_margin 0.102)
 		)

Commit message: 製造ファイル再生成
Parts:
- moved C30 0.35 mm to (-0.75, 13.5)
- moved C5 0.35 mm to (0.75, 12.0)
Routing:
- net GND: vias 227 -> 242
Other:
- board text added: "CLK"
- board text added: "DIO"
- board text added: "GND"
- board text added: "NSRT"
